Commit message: gazebo position control plugin working

File: sbot_description/urdf/macros_links_y_joints.xacro (robot description, xacro)
@@ -15,4 +15,5 @@
   <xacro:macro name="m_link" params="name color origin_xyz origin_rpy meshfile meshscale mass ixx ixy ixz iyy iyz izz">
     <link name="${name}">
+      <!-- <selfCollide>true</selfCollide> -->
       <inertial>
         <mass value="${mass}" />

File: sbot_description/urdf/sbot_arm.urdf.xacro (robot description, xacro)
@@ -152,10 +152,10 @@
     <!-- DEFINO EE_LINK -->
     <link name="ee_link">
-      <collision>
+      <!-- <collision>
         <geometry>
           <box size="0.001 0.001 0.001"/>
         </geometry>
         <origin rpy="0 0 0" xyz="-0.01 0 0"/>
-      </collision>
+      </collision> -->
     </link>
     <!-- DEFINO EE_FIXED_JOINT -->

File: sbot_gazebo/config/sbot.urdf.xacro (robot description, xacro)
@@ -1,13 +1,14 @@
 <?xml version="1.0"?>
-<robot xmlns:xacro="http://www.ros.org/wiki/xacro" name="sbot">
+<robot xmlns:xacro="http://www.ros.org/wiki/xacro" name="scorbot">
     <!-- Import sbot urdf file -->
-    <!-- <xacro:include filename="$(find sbot_description)/urdf/scorbot.urdf.xacro" /> -->
+    <xacro:include filename="$(find sbot_description)/urdf/scorbot.urdf.xacro" />
     <!-- Import control_xacro -->
-    <xacro:include filename="transmission_gazebo.xacro" />
+    <!-- <xacro:include filename="transmission_gazebo.xacro" /> -->
       <!-- JOINT PUBLISHER -->
   <gazebo>
+   <self_collide>true</self_collide>
     <plugin filename="ignition-gazebo-joint-state-publisher-system" name="gz::sim::systems::JointStatePublisher">
       <ros>
-        <remapping>~/out:=sbot/joint_states</remapping>
+        <remapping>~/out:=scorbot/joint_states</remapping>
       </ros>
       <update_rate>30</update_rate>
@@ -20,13 +21,13 @@
       <joint_name>roll</joint_name>
     </plugin>
-        <xacro:macro name="joint_position_controller" params="joint_name p_gain:=1 d_gain:=0 i_gain:=0 mimic_joint:=''">
+    <xacro:macro name="joint_position_controller" params="joint_name p_gain:=1 d_gain:=0 i_gain:=0 mimic_joint:=''">
       <plugin filename="ignition-gazebo-joint-position-controller-system"
         name="gz::sim::systems::JointPositionController">
-        <!-- <xacro:if value="${mimic_joint == ''}">
+        <xacro:if value="${mimic_joint == ''}">
           <xacro:property name="topic_joint" value="${joint_name}"/>
         </xacro:if>
         <xacro:unless value="${mimic_joint == ''}">
           <xacro:property name="topic_joint" value="${mimic_joint}"/>
-        </xacro:unless> -->
+        </xacro:unless>
         <joint_name>${joint_name}</joint_name>
         <p_gain>${p_gain}</p_gain>
@@ -35,5 +36,5 @@
         <i_max>1000</i_max>
         <i_min>-1000</i_min>
-        <topic>/model/scorbot/joint/${joint_name}/cmd_pos</topic>
+        <topic>/model/scorbot/joint/${topic_joint}/cmd_pos</topic>
       </plugin>
     </xacro:macro>
@@ -43,5 +44,5 @@
     <xacro:joint_position_controller joint_name="pitch" p_gain="1e4" d_gain="1e1" i_gain="1e1"/>
     <xacro:joint_position_controller joint_name="roll" p_gain="1e4" d_gain="1e1" i_gain="1e1"/>
-    <xacro:joint_position_controller joint_name="finger_R_joint" p_gain="1e4" d_gain="1e1" i_gain="1e1"/>
+    <xacro:joint_position_controller joint_name="finger_R_joint" p_gain="1e4" d_gain="1e1" i_gain="1e1" mimic_joint="finger_L_joint"/>
     <xacro:joint_position_controller joint_name="finger_L_joint" p_gain="1e4" d_gain="1e" i_gain="1e1"/>
   </gazebo>
