Commit message: modificaciones modulares

File: sbot_description/urdf/sbot_arm.urdf.xacro (robot description, xacro)
@@ -11,5 +11,5 @@
   Author: Felix Messmer
 -->
-  <xacro:macro name="sbot_arm" params="prefix joint_limited shoulder_pan_lower_limit:=${-pi} shoulder_pan_upper_limit:=${pi} shoulder_lift_lower_limit:=${-pi} shoulder_lift_upper_limit:=${pi} elbow_joint_lower_limit:=${-pi} elbow_joint_upper_limit:=${pi} wrist_1_lower_limit:=${-pi} wrist_1_upper_limit:=${pi} wrist_2_lower_limit:=${-pi} wrist_2_upper_limit:=${pi} wrist_3_lower_limit:=${-pi} wrist_3_upper_limit:=${pi} transmission_hw_interface:=hardware_interface/PositionJointInterface safety_limits:=false safety_pos_margin:=0.15 safety_k_position:=20">
+  <xacro:macro name="sbot_arm" params="prefix joint_limited">
     <!-- LINKS REALES DEL BRAZO -->
     <xacro:property name="robot_name" default="scorbot"/>
@@ -31,13 +31,104 @@
     <xacro:property name="forearm_mass" value="5.6889976191393" />
     <xacro:property name="flange_mass" value="1.08471916910904" />
-    <xacro:m_link name="${base}" color="Grey" origin_rpy="0 0 0" origin_xyz="-0.108054021244931 -6.78949721999444E-08 0.0484049851585737" mass="${base_mass}" ixx="0.085126670768749" ixy="2.58404334129752E-08" ixz="-1.08844213882229E-08" iyy="0.085126691797693" iyz="-6.7077388590106E-09" izz="0.0998601414904193" meshfile="file:$(find sbot_description)/meshes/link_base.STL" meshscale="1 1 1" />
-    <xacro:m_link name="${body}" color="Grey" origin_rpy="0 0 0" origin_xyz="-0.0593135451515788 -0.00322725876445507 0.320154858954509" mass="${body_mass}" ixx="0.145932144728803" ixy="0.00612026711691293" ixz="-0.0110238426104326" iyy="0.254113528367173" iyz="0.00247600075693871" izz="0.247916599392411" meshfile="file:$(find sbot_description)/meshes/link_one.STL" meshscale="1 1 1" />
-    <xacro:m_link name="${upper_arm}" color="Grey" origin_rpy="0 0 0" origin_xyz="4.85332329874938E-05 0.0339669542339676 0.1583205027378" mass="${upper_arm_mass}" ixx="0.145932144728803" ixy="0.00612026711691293" ixz="-0.0110238426104326" iyy="0.254113528367173" iyz="0.00247600075693871" izz="0.247916599392411" meshfile="file:$(find sbot_description)/meshes/link_two.STL" meshscale="1 1 1" />
-    <xacro:m_link name="${forearm}" color="Grey" origin_rpy="0 0 0" origin_xyz="-1.47432084651733E-07 -0.111132038571227 0.0375927278081665" mass="${forearm_mass}" ixx="0.066293063521651" ixy="-6.29583836298716E-08" ixz="-5.35286377624852E-08" iyy="0.012551076830058" iyz="-0.000390405491272255" izz="0.0629744677227373" meshfile="file:$(find sbot_description)/meshes/link_three.STL" meshscale="1 1 1" />
-    <xacro:m_link name="${flange}" color="Grey" origin_rpy="0 0 0" origin_xyz="-0.0382603821035229 -0.00311385230179761 0.0369189530731333" mass="${flange_mass}" ixx="0.000700705072423402" ixy="0.000134315224988601" ixz="3.57613195744678E-06" iyy="0.0024076862804167" iyz="-2.44981684573351E-07" izz="0.00265552184192292" meshfile="file:$(find sbot_description)/meshes/link_four.STL" meshscale="1 1 1" />
-    <xacro:m_joint name="${base_joint}" type="continuous" axis_xyz="0 0 -1" origin_rpy="0 0 0" origin_xyz="-0.10805388876492 0 0" parent="${base}" child="${body}" limit_e="1000" limit_l="-2.3562" limit_u="2.3562" limit_v="0.5" />
-    <xacro:m_joint name="${elbow}" type="continuous" axis_xyz="0 0 1" origin_rpy="1.5708 0 0" origin_xyz="0.07 0 0.372" parent="${body}" child="${upper_arm}" limit_e="1000" limit_l="-2.3562" limit_u="2.3562" limit_v="0.5" />
-    <xacro:m_joint name="${shoulder}" type="continuous" axis_xyz="0 0 1" origin_rpy="0 0 1.5708" origin_xyz="0 0.28 0" parent="${upper_arm}" child="${forearm}" limit_e="1000" limit_l="-2.3562" limit_u="2.3562" limit_v="0.5" />
-    <xacro:m_joint name="${pitch}" type="continuous" axis_xyz="0 0 1" origin_rpy="0 0 -1.5708" origin_xyz="0 -0.23 0" parent="${forearm}" child="${flange}" limit_e="1000" limit_l="-2.3562" limit_u="2.3562" limit_v="0.5" />
+    <xacro:m_link name="${base}" color="Grey"
+            origin_rpy="0 0 0"
+            origin_xyz="-0.108054021244931 -6.78949721999444E-08 0.0484049851585737"
+            mass="${base_mass}"
+            ixx="0.085126670768749"
+            ixy="2.58404334129752E-08"
+            ixz="-1.08844213882229E-08"
+            iyy="0.085126691797693"
+            iyz="-6.7077388590106E-09"
+            izz="0.0998601414904193"
+            meshfile="file:$(find sbot_description)/meshes/link_base.STL"
+            meshscale="1 1 1" />
+    <xacro:m_link name="${body}" color="Grey"
+            origin_rpy="0 0 0"
+            origin_xyz="-0.0593135451515788 -0.00322725876445507 0.320154858954509"
+            mass="${body_mass}"
+            ixx="0.145932144728803"
+            ixy="0.00612026711691293"
+            ixz="-0.0110238426104326"
+            iyy="0.254113528367173"
+            iyz="0.00247600075693871"
+            izz="0.247916599392411"
+            meshfile="file:$(find sbot_description)/meshes/link_one.STL"
+            meshscale="1 1 1" />
+    <xacro:m_link name="${upper_arm}" color="Grey"
+                origin_rpy="0 0 0"
+                origin_xyz="4.85332329874938E-05 0.0339669542339676 0.1583205027378"
+                mass="${upper_arm_mass}"
+                ixx="0.145932144728803"
+                ixy="0.00612026711691293"
+                ixz="-0.0110238426104326"
+                iyy="0.254113528367173"
+                iyz="0.00247600075693871"
+                izz="0.247916599392411"
+                meshfile="file:$(find sbot_description)/meshes/link_two.STL"
+                meshscale="1 1 1" />
+    <xacro:m_link name="${forearm}" color="Grey"
+                origin_rpy="0 0 0"
+                origin_xyz="-1.47432084651733E-07 -0.111132038571227 0.0375927278081665"
+                mass="${forearm_mass}"
+                ixx="0.066293063521651"
+                ixy="-6.29583836298716E-08"
+                ixz="-5.35286377624852E-08"
+                iyy="0.012551076830058"
+                iyz="-0.000390405491272255"
+                izz="0.0629744677227373"
+                meshfile="file:$(find sbot_description)/meshes/link_three.STL"
+                meshscale="1 1 1" />
+    <xacro:m_link name="${flange}" color="Grey"
+                origin_rpy="0 0 0"
+                origin_xyz="-0.0382603821035229 -0.00311385230179761 0.0369189530731333"
+                mass="${flange_mass}"
+                ixx="0.000700705072423402"
+                ixy="0.000134315224988601"
+                ixz="3.57613195744678E-06"
+                iyy="0.0024076862804167"
+                iyz="-2.44981684573351E-07"
+                izz="0.00265552184192292"
+                meshfile="file:$(find sbot_description)/meshes/link_four.STL"
+                meshscale="1 1 1" />
+    <xacro:m_joint name="${base_joint}" type="continuous"
+                axis_xyz="0 0 -1"
+                origin_rpy="0 0 0"
+                origin_xyz="-0.10805388876492 0 0"
+                parent="${base}"
+                child="${body}"
+                limit_e="1000"
+                limit_l="-2.3562"
+                limit_u="2.3562"
+                limit_v="0.5" />
+    <xacro:m_joint name="${elbow}" type="continuous"
+                axis_xyz="0 0 1"
+                origin_rpy="1.5708 0 0"
+                origin_xyz="0.07 0 0.372"
+                parent="${body}"
+                child="${upper_arm}"
+                limit_e="1000"
+                limit_l="-2.3562"
+                limit_u="2.3562"
+                limit_v="0.5" />
+    <xacro:m_joint name="${shoulder}" type="continuous"
+                axis_xyz="0 0 1"
+                origin_rpy="0 0 1.5708"
+                origin_xyz="0 0.28 0"
+                parent="${upper_arm}"
+                child="${forearm}"
+                limit_e="1000"
+                limit_l="-2.3562"
+                limit_u="2.3562"
+                limit_v="0.5" />
+    <xacro:m_joint name="${pitch}" type="continuous"
+                axis_xyz="0 0 1"
+                origin_rpy="0 0 -1.5708"
+                origin_xyz="0 -0.23 0"
+                parent="${forearm}"
+                child="${flange}"
+                limit_e="1000"
+                limit_l="-2.3562"
+                limit_u="2.3562"
+                limit_v="0.5" />
     <!-- DEFINO UN CILINDRO INTERMEDIO PARA QUE GIRE EL GRIPPER LUEGO -->
     <link name="cylinder_link">

File: sbot_description/urdf/sbot_gripper.urdf.xacro (robot description, xacro)
@@ -70,5 +70,5 @@
                     origin_rpy="-1.5708 0 0" origin_xyz="0 0 0.134"
                     parent="${gripper}" child="${finger_R}"
-                    limit_e="1000" limit_l="0" limit_u="0.024" limit_v="0.5" mimic="true"
+                    limit_e="1000" limit_l="0" limit_u="0.02" limit_v="0.5" mimic="true"
                     />
     </xacro:macro>

File: sbot_description/urdf/scorbot.urdf.xacro (robot description, xacro)
@@ -9,4 +9,5 @@
     <!-- GENERAR EL BRAZO -->
     <xacro:sbot_arm prefix="" joint_limited="false"/>
+    <!-- joint limited no se uso -->
     <link name="world"/>
     <joint name="world_joint" type="fixed">
@@ -21,48 +22,6 @@
     <!-- Gazebo stuff -->
     <xacro:include filename="$(find sbot_description)/urdf/physical_properties.xacro" />
-    <xacro:include filename="$(find sbot_description)/urdf/transmission_gazebo.xacro" />
     <!-- Control stuff -->
     <!-- <xacro:include filename="$(find sbot_description)/urdf/ros2control.xacro" /> -->
   <!-- PLUGINS -->
-  <!-- JOINT PUBLISHER -->
-  <gazebo>
-    <plugin filename="ignition-gazebo-joint-state-publisher-system" name="gz::sim::systems::JointStatePublisher">
-      <ros>
-        <remapping>~/out:=sbot/joint_states</remapping>
-      </ros>
-      <update_rate>30</update_rate>
-      <joint_name>finger_R_joint</joint_name>
-      <joint_name>finger_L_joint</joint_name>
-      <joint_name>base_joint</joint_name>
-      <joint_name>elbow</joint_name>
-      <joint_name>shoulder</joint_name>
-      <joint_name>pitch</joint_name>
-      <joint_name>roll</joint_name>
-    </plugin>
-    <xacro:macro name="joint_position_controller" params="joint_name p_gain:=1 d_gain:=0 i_gain:=0 mimic_joint:=''">
-      <plugin filename="ignition-gazebo-joint-position-controller-system"
-        name="gz::sim::systems::JointPositionController">
-        <!-- <xacro:if value="${mimic_joint == ''}">
-          <xacro:property name="topic_joint" value="${joint_name}"/>
-        </xacro:if>
-        <xacro:unless value="${mimic_joint == ''}">
-          <xacro:property name="topic_joint" value="${mimic_joint}"/>
-        </xacro:unless> -->
-        <joint_name>${joint_name}</joint_name>
-        <p_gain>${p_gain}</p_gain>
-        <d_gain>${d_gain}</d_gain>
-        <i_gain>${i_gain}</i_gain>
-        <i_max>1000</i_max>
-        <i_min>-1000</i_min>
-        <topic>/model/scorbot/joint/${joint_name}/cmd_pos</topic>
-      </plugin>
-    </xacro:macro>
-    <xacro:joint_position_controller joint_name="base_joint" p_gain="1e4" d_gain="1e1" i_gain="1e1"/>
-    <xacro:joint_position_controller joint_name="elbow" p_gain="1e4" d_gain="1e1" i_gain="1e1"/>
-    <xacro:joint_position_controller joint_name="shoulder" p_gain="1e4" d_gain="1e1" i_gain="1e1"/>
-    <xacro:joint_position_controller joint_name="pitch" p_gain="1e4" d_gain="1e1" i_gain="1e1"/>
-    <xacro:joint_position_controller joint_name="roll" p_gain="1e4" d_gain="1e1" i_gain="1e1"/>
-    <xacro:joint_position_controller joint_name="finger_R_joint" p_gain="1e4" d_gain="1e1" i_gain="1e1"/>
-    <xacro:joint_position_controller joint_name="finger_L_joint" p_gain="1e4" d_gain="1e" i_gain="1e1"/>
- </gazebo>
 </robot>

Commit message: Delete cylinder collision, gazebo collsion works

File: sbot_description/urdf/sbot_arm.urdf.xacro (robot description, xacro)
@@ -142,10 +142,10 @@
         </material>
       </visual>
-      <collision>
+      <!-- <collision>
         <origin xyz="0 0 0" rpy="0 0 0" />
         <geometry>
           <cylinder radius="0.01" length="0.05" />
         </geometry>
-      </collision>
+      </collision> -->
     </link>
     <xacro:m_joint name="${roll}" type="continuous" axis_xyz="0 0 -1" origin_rpy="-1.5708 0 -1.5708" origin_xyz="0 -0.0058721 0.036836" parent="${flange}" child="cylinder_link" limit_e="1000" limit_l="-2.3562" limit_u="2.3562" limit_v="0.5" />

Commit message: sbot desc y sbot gazebo modificados

File: sbot_description/urdf/sbot_arm.urdf.xacro (robot description, xacro)
@@ -21,6 +21,6 @@
     <!-- JUNTAS REALES DEL BRAZO -->
     <xacro:property name="base_joint" default="base_joint"/>
+    <xacro:property name="shoulder" default="shoulder"/>
     <xacro:property name="elbow" default="elbow"/>
-    <xacro:property name="shoulder" default="shoulder"/>
     <xacro:property name="pitch" default="pitch"/>
     <xacro:property name="roll" default="roll"/>
@@ -101,5 +101,6 @@
                 limit_u="2.3562"
                 limit_v="0.5" />
-    <xacro:m_joint name="${elbow}" type="continuous"
+<!-- cambie el shoulder por el elbow -->
+    <xacro:m_joint name="${shoulder}" type="continuous"
                 axis_xyz="0 0 1"
                 origin_rpy="1.5708 0 0"
@@ -111,5 +112,5 @@
                 limit_u="2.3562"
                 limit_v="0.5" />
-    <xacro:m_joint name="${shoulder}" type="continuous"
+    <xacro:m_joint name="${elbow}" type="continuous"
                 axis_xyz="0 0 1"
                 origin_rpy="0 0 1.5708"

File: sbot_gazebo/config/gz_ros2_control.xacro (robot description, xacro)
@@ -1,16 +1,175 @@
 <?xml version="1.0"?>
 <robot xmlns:xacro="http://www.ros.org/wiki/xacro" name="scorbot">
+<!-- transmision tags to add versatility in gazebo are not required to ros control works -->
+        <!-- base_joint -->
+        <transmission name="trans_base_joint">
+            <type>transmission_interface/SimpleTransmission</type>
+            <joint name="base_joint">
+                <hardwareInterface>hardware_interface/PositionJointInterface</hardwareInterface>
+            </joint>
+            <actuator name="motor_base_joint">
+                <hardwareInterface>hardware_interface/PositionJointInterface</hardwareInterface>
+                <mechanicalReduction>1</mechanicalReduction>
+            </actuator>
+        </transmission>
+        <!-- elbow -->
+        <transmission name="trans_elbow">
+            <type>transmission_interface/SimpleTransmission</type>
+            <joint name="elbow">
+                <hardwareInterface>hardware_interface/PositionJointInterface</hardwareInterface>
+            </joint>
+            <actuator name="motor_elbow">
+                <hardwareInterface>hardware_interface/PositionJointInterface</hardwareInterface>
+                <mechanicalReduction>1</mechanicalReduction>
+            </actuator>
+        </transmission>
+        <!-- shoulder -->
+        <transmission name="trans_shoulder">
+            <type>transmission_interface/SimpleTransmission</type>
+            <joint name="shoulder">
+                <hardwareInterface>hardware_interface/PositionJointInterface</hardwareInterface>
+            </joint>
+            <actuator name="motor_shoulder">
+                <hardwareInterface>hardware_interface/PositionJointInterface</hardwareInterface>
+                <mechanicalReduction>1</mechanicalReduction>
+            </actuator>
+        </transmission>
+        <!-- pitch -->
+        <transmission name="trans_pitch">
+            <type>transmission_interface/SimpleTransmission</type>
+            <joint name="pitch">
+                <hardwareInterface>hardware_interface/PositionJointInterface</hardwareInterface>
+            </joint>
+            <actuator name="motor_pitch">
+                <hardwareInterface>hardware_interface/PositionJointInterface</hardwareInterface>
+                <mechanicalReduction>1</mechanicalReduction>
+            </actuator>
+        </transmission>
+        <!-- roll -->
+        <transmission name="trans_roll">
+            <type>transmission_interface/SimpleTransmission</type>
+            <joint name="roll">
+                <hardwareInterface>hardware_interface/PositionJointInterface</hardwareInterface>
+            </joint>
+            <actuator name="motor_roll">
+                <hardwareInterface>hardware_interface/PositionJointInterface</hardwareInterface>
+                <mechanicalReduction>1</mechanicalReduction>
+            </actuator>
+        </transmission>
+        <!-- finger_R_joint -->
+        <!-- <transmission name="trans_finger_R_joint">
+            <type>transmission_interface/SimpleTransmission</type>
+            <joint name="finger_R_joint">
+                <hardwareInterface>hardware_interface/PositionJointInterface</hardwareInterface>
+            </joint>
+            <actuator name="motor_finger_R_joint">
+                <hardwareInterface>hardware_interface/PositionJointInterface</hardwareInterface>
+                <mechanicalReduction>1</mechanicalReduction>
+            </actuator>
+        </transmission> -->
+        <!-- <xacro:macro name="mimic_joint_plugin_ignition" params="parent_joint mimic_joint has_pid:=false multiplier:=1.0 offset:=0 sensitiveness:=0.0 max_effort:=200.0 robot_namespace:=''">
+            <gazebo>
+                <plugin name="${mimic_joint}_mimic_joint_plugin" filename="libroboticsgroup_ignition_mimic_joint_plugin.so">
+                    <joint>${parent_joint}</joint>
+                    <mimicJoint>${mimic_joint}</mimicJoint>
+                    <xacro:if value="${has_pid}">
+                    <hasPID />
+                    </xacro:if>
+                    <multiplier>${multiplier}</multiplier>
+                    <offset>${offset}</offset>
+                    <sensitiveness>${sensitiveness}</sensitiveness>
+                    <maxEffort>${max_effort}</maxEffort>
+                    <xacro:unless value="${robot_namespace == ''}">
+                        <robotNamespace>($robot_namespace)</robotNamespace>
+                    </xacro:unless>
+                </plugin>
+            </gazebo>
+        </xacro:macro> -->
+        <!-- <xacro:mimic_joint_plugin_ignition parent_joint="finger_L_joint"
+        mimic_joint="finger_R_joint" has_pid="false" multiplier="1.0"
+        max_effort="200.0" /> -->
+        <!-- finger_L_joint -->
+        <transmission name="trans_finger_L_joint">
+            <type>transmission_interface/SimpleTransmission</type>
+            <joint name="finger_L_joint">
+                <hardwareInterface>hardware_interface/PositionJointInterface</hardwareInterface>
+            </joint>
+            <actuator name="motor_finger_L_joint">
+                <hardwareInterface>hardware_interface/PositionJointInterface</hardwareInterface>
+                <mechanicalReduction>1</mechanicalReduction>
+            </actuator>
+        </transmission>
     <!-- Argumentos de ros2_control sobre gazebo -->
     <!-- Posiciones iniciales de las juntas -->
     <xacro:arg name="initial_positions_file" default="initial_positions.yaml" />
-    <!-- Import control_xacro -->
-    <xacro:include filename="scorbot.ros2_control.xacro" />
+    <!-- Import ros2_control_xacro -->
+    <!-- <xacro:include filename="scorbot.ros2_control.xacro" /> -->
+    <!-- creo que es mejor tener todo en este archivo antes que importar la linea anterior -->
+        <xacro:macro name="scorbot_ros2_control" params="name initial_positions_file">
+        <xacro:property name="initial_positions" value="${xacro.load_yaml(initial_positions_file)['initial_positions']}"/>
+        <!-- definiciones de ros2 control para el control de las juntas -->
+        <ros2_control name="${name}" type="system">
+            <hardware>
+                <!-- By default, set up controllers for simulation. This won't work on real hardware -->
+                <!-- para visualizacion  -->
+                <!-- <plugin>mock_components/GenericSystem</plugin> -->
+                <!-- para simulacion en gazebo -->
+                <plugin>ign_ros2_control/IgnitionSystem</plugin>
+                <!-- para control en sistema real -->
+                <!-- <plugin>ign_ros2_control/IgnitionSystem</plugin> -->
+            </hardware>
+            <joint name="base_joint">
+                <command_interface name="position"/>
+                <state_interface name="position">
+                  <param name="initial_value">${initial_positions['base_joint']}</param>
+                </state_interface>
+                <state_interface name="velocity"/>
+            </joint>
+            <joint name="shoulder">
+                <command_interface name="position"/>
+                <state_interface name="position">
+                  <param name="initial_value">${initial_positions['shoulder']}</param>
+                </state_interface>
+                <state_interface name="velocity"/>
+            </joint>
+            <joint name="elbow">
+                <command_interface name="position"/>
+                <state_interface name="position">
+                  <param name="initial_value">${initial_positions['elbow']}</param>
+                </state_interface>
+                <state_interface name="velocity"/>
+            </joint>
+            <joint name="pitch">
+                <command_interface name="position"/>
+                <state_interface name="position">
+                  <param name="initial_value">${initial_positions['pitch']}</param>
+                </state_interface>
+                <state_interface name="velocity"/>
+            </joint>
+            <joint name="roll">
+                <command_interface name="position"/>
+                <state_interface name="position">
+                  <param name="initial_value">${initial_positions['roll']}</param>
+                </state_interface>
+                <state_interface name="velocity"/>
+            </joint>
+            <joint name="finger_L_joint">
+                <command_interface name="position"/>
+                <state_interface name="position">
+                  <param name="initial_value">${initial_positions['finger_L_joint']}</param>
+                </state_interface>
+                <state_interface name="velocity"/>
+            </joint>
+        </ros2_control>
+    </xacro:macro>
     <xacro:scorbot_ros2_control name="IgnitionSystem" initial_positions_file="$(arg initial_positions_file)"/>
     <gazebo>
-    <!-- Plugin de gazebo sobre ros2_control -->
+        <!-- Plugin de gazebo sobre ros2_control -->
         <plugin filename="ign_ros2_control-system" name="ign_ros2_control::IgnitionROS2ControlPlugin">
                 <robot_param>/robot_description</robot_param>
                 <parameters>$(find sbot_moveit_gz)/config/ros2_controllers.yaml</parameters>
                 <robot_param_node>/robot_state_publisher</robot_param_node>
+                <!-- AÑADIDO A CHEQUEAR -->
+                <!-- <parameters>$(find my_package)/config/my_joint_state_broadcaster.yaml</parameters> -->
         </plugin>
     </gazebo>
