Commit message: moveit_nuevo

File: sbot_description/urdf/sbot_arm.urdf.xacro (robot description, xacro)
@@ -91,5 +91,5 @@
                 meshfile="file:$(find sbot_description)/meshes/link_four.STL"
                 meshscale="1 1 1" />
-    <xacro:m_joint name="${base_joint}" type="continuous"
+    <xacro:m_joint name="${base_joint}" type="revolute"
                 axis_xyz="0 0 -1"
                 origin_rpy="0 0 0"
@@ -102,5 +102,5 @@
                 limit_v="0.5" />
 <!-- cambie el shoulder por el elbow -->
-    <xacro:m_joint name="${shoulder}" type="continuous"
+    <xacro:m_joint name="${shoulder}" type="revolute"
                 axis_xyz="0 0 1"
                 origin_rpy="1.5708 0 0"
@@ -112,5 +112,5 @@
                 limit_u="2.3562"
                 limit_v="0.5" />
-    <xacro:m_joint name="${elbow}" type="continuous"
+    <xacro:m_joint name="${elbow}" type="revolute"
                 axis_xyz="0 0 1"
                 origin_rpy="0 0 1.5708"
@@ -122,5 +122,5 @@
                 limit_u="2.3562"
                 limit_v="0.5" />
-    <xacro:m_joint name="${pitch}" type="continuous"
+    <xacro:m_joint name="${pitch}" type="revolute"
                 axis_xyz="0 0 1"
                 origin_rpy="0 0 -1.5708"

File: sbot_gazebo/config/scorbot_gz.urdf.xacro (robot description, xacro)
@@ -1,5 +1,5 @@
 <?xml version="1.0"?>
 <robot xmlns:xacro="http://www.ros.org/wiki/xacro" name="scorbot">
-<!-- Archivo de control para simulacion  -->
+    <!-- Archivo de control para simulacion  -->
     <!-- Import sbot urdf file -->
     <xacro:include filename="$(find sbot_description)/urdf/scorbot.urdf.xacro" />

File: sbot_moveit/config/scorbot.ros2_control.xacro (robot description, xacro)
@@ -1,10 +1,10 @@
 <?xml version="1.0"?>
 <robot xmlns:xacro="http://www.ros.org/wiki/xacro">
-    <xacro:macro name="scorbot_ros2_control" params="name initial_positions_file system">
+    <xacro:macro name="scorbot_ros2_control" params="name initial_positions_file">
         <xacro:property name="initial_positions" value="${load_yaml(initial_positions_file)['initial_positions']}"/>
         <ros2_control name="${name}" type="system">
             <hardware>
                 <!-- By default, set up controllers for simulation. This won't work on real hardware -->
-                <plugin>"${system}"</plugin>
+                <plugin>mock_components/GenericSystem</plugin>
             </hardware>
             <joint name="base_joint">
@@ -15,15 +15,15 @@
                 <state_interface name="velocity"/>
             </joint>
+            <joint name="shoulder">
+                <command_interface name="position"/>
+                <state_interface name="position">
+                  <param name="initial_value">${initial_positions['shoulder']}</param>
+                </state_interface>
+                <state_interface name="velocity"/>
+            </joint>
             <joint name="elbow">
                 <command_interface name="position"/>
                 <state_interface name="position">
                   <param name="initial_value">${initial_positions['elbow']}</param>
-                </state_interface>
-                <state_interface name="velocity"/>
-            </joint>
-            <joint name="shoulder">
-                <command_interface name="position"/>
-                <state_interface name="position">
-                  <param name="initial_value">${initial_positions['shoulder']}</param>
                 </state_interface>
                 <state_interface name="velocity"/>

File: sbot_moveit/config/scorbot.urdf.xacro (robot description, xacro)
@@ -1,21 +1,9 @@
 <?xml version="1.0"?>
 <robot xmlns:xacro="http://www.ros.org/wiki/xacro" name="scorbot">
-    <!-- <arg name="sim_gazebo"            default="False"/>
-    <arg name="no_sim_gazebo"         default="True"/> -->
     <xacro:arg name="initial_positions_file" default="initial_positions.yaml" />
     <!-- Import scorbot urdf file -->
     <xacro:include filename="$(find sbot_description)/urdf/scorbot.urdf.xacro" />
+    <!-- Import control_xacro -->
     <xacro:include filename="scorbot.ros2_control.xacro" />
-    <!-- <include if="$(arg sim_gazebo)">
-        <xacro:scorbot_ros2_control name="IgnSystem"
-        system="ign_ros2_control/IgnitionSystem"
-        initial_positions_file="$(arg initial_positions_file)"/>
-    </include> -->
-    <!-- <include if="$(arg no_sim_gazebo)"> -->
-     <include>
-        <!-- Import control_xacro -->
-        <xacro:scorbot_ros2_control name="FakeSystem"
-        system="mock_components/GenericSystem"
-        initial_positions_file="$(arg initial_positions_file)"/>
-    </include>
+    <xacro:scorbot_ros2_control name="FakeSystem" initial_positions_file="$(arg initial_positions_file)"/>
 </robot>

Commit message: demo -] moveit

File: sbot_description/urdf/sbot_arm.urdf.xacro (robot description, xacro)
@@ -150,5 +150,14 @@
       </collision> -->
     </link>
-    <xacro:m_joint name="${roll}" type="continuous" axis_xyz="0 0 -1" origin_rpy="-1.5708 0 -1.5708" origin_xyz="0 -0.0058721 0.036836" parent="${flange}" child="cylinder_link" limit_e="1000" limit_l="-2.3562" limit_u="2.3562" limit_v="0.5" />
+    <xacro:m_joint name="${roll}" type="continuous"
+                  axis_xyz="0 0 -1"
+                  origin_rpy="-1.5708 0 -1.5708"
+                  origin_xyz="0 -0.0058721 0.036836"
+                  parent="${flange}"
+                  child="cylinder_link"
+                  limit_e="1000"
+                  limit_l="-2.3562"
+                  limit_u="2.3562"
+                  limit_v="0.5" />
     <!-- DEFINO EE_LINK -->
     <link name="ee_link">

File: sbot_moveit/config/scorbot.ros2_control.xacro (robot description, xacro)
@@ -1,10 +1,9 @@
 <?xml version="1.0"?>
 <robot xmlns:xacro="http://www.ros.org/wiki/xacro">
-    <xacro:macro name="scorbot_ros2_control" params="name initial_positions_file">
+    <xacro:macro name="scorbot_ros2_control" params="name initial_positions_file system">
         <xacro:property name="initial_positions" value="${load_yaml(initial_positions_file)['initial_positions']}"/>
         <ros2_control name="${name}" type="system">
             <hardware>
-                <!-- By default, set up controllers for simulation. This won't work on real hardware -->
-                <plugin>mock_components/GenericSystem</plugin>
+              <plugin>${system}</plugin>
             </hardware>
             <joint name="base_joint">
@@ -52,3 +51,11 @@
         </ros2_control>
     </xacro:macro>
+    <gazebo>
+        <!-- Plugin de gazebo sobre ros2_control -->
+        <plugin filename="ign_ros2_control-system" name="ign_ros2_control::IgnitionROS2ControlPlugin">
+                <robot_param>/robot_description</robot_param>
+                <parameters>$(find sbot_moveit)/config/ros2_controllers.yaml</parameters>
+                <robot_param_node>/robot_state_publisher</robot_param_node>
+        </plugin>
+    </gazebo>
 </robot>

File: sbot_moveit/config/scorbot.urdf.xacro (robot description, xacro)
@@ -2,8 +2,15 @@
 <robot xmlns:xacro="http://www.ros.org/wiki/xacro" name="scorbot">
     <xacro:arg name="initial_positions_file" default="initial_positions.yaml" />
+    <!-- <xacro:arg name="sim_gz" type="bool" default="false"/> -->
+    <xacro:arg name="fake" type="bool" default="false"/>
     <!-- Import scorbot urdf file -->
     <xacro:include filename="$(find sbot_description)/urdf/scorbot.urdf.xacro" />
     <!-- Import control_xacro -->
     <xacro:include filename="scorbot.ros2_control.xacro" />
-    <xacro:scorbot_ros2_control name="FakeSystem" initial_positions_file="$(arg initial_positions_file)"/>
+    <!-- <include if="$(arg fake)"> -->
+    <xacro:scorbot_ros2_control name="FakeSystem" system="mock_components/GenericSystem"  initial_positions_file="$(arg initial_positions_file)"/>
+    <!-- </include> -->
+    <!-- <xacro:if value="$(arg sim_gz)">
+        <xacro:scorbot_ros2_control name="IgnitionSystem" system="ign_ros2_control/IgnitionSystem" initial_positions_file="$(arg initial_positions_file)"/>
+    </xacro:if>  -->
 </robot>

Commit message: sbot y sbot gazebo + modificacione ee_link

File: sbot_description/urdf/sbot_arm.urdf.xacro (robot description, xacro)
@@ -173,5 +173,6 @@
       <parent link="cylinder_link" />
       <child link = "ee_link" />
-      <origin xyz="0.0 0.0 0.0" rpy="0.0 0.0 0.0" />
+      <origin xyz="0 0 0.170" rpy="0.0 0.0 0.0" />
+      <!-- cambie por el 0 0 0 para llevar el end effector mas adelante -->
     </joint>
     <!--0.123619254184439-->

File: sbot_moveit _gazebo/config/scorbot.ros2_control.xacro (robot description, xacro)
@@ -5,5 +5,6 @@
         <ros2_control name="${name}" type="system">
             <hardware>
-              <plugin>${system}</plugin>
+                <!-- By default, set up controllers for simulation. This won't work on real hardware -->
+                <plugin>${system}</plugin>
             </hardware>
             <joint name="base_joint">

File: sbot_moveit _gazebo/config/scorbot.urdf.xacro (robot description, xacro)
@@ -5,5 +5,5 @@
     <xacro:include filename="$(find sbot_description)/urdf/scorbot.urdf.xacro" />
     <!-- Import control_xacro -->
-    <xacro:include filename="scorbot_gz.ros2_control.xacro" />
+    <xacro:include filename="scorbot.ros2_control.xacro" />
     <!-- Macro control_xacro -->
     <xacro:scorbot_ros2_control name="IgnitionSystem" system="ign_ros2_control/IgnitionSystem" initial_positions_file="$(arg initial_positions_file)"/>

File: sbot_moveit/config/scorbot.ros2_control.xacro (robot description, xacro)
@@ -5,5 +5,6 @@
         <ros2_control name="${name}" type="system">
             <hardware>
-              <plugin>${system}</plugin>
+                <!-- By default, set up controllers for simulation. This won't work on real hardware -->
+                <plugin>${system}</plugin>
             </hardware>
             <joint name="base_joint">
@@ -51,11 +52,3 @@
         </ros2_control>
     </xacro:macro>
-    <!-- Plugin de gazebo sobre ros2_control -->
-    <!-- <gazebo>
-        <plugin filename="ign_ros2_control-system" name="ign_ros2_control::IgnitionROS2ControlPlugin">
-                <robot_param>/robot_description</robot_param>
-                <parameters>$(find sbot_moveit)/config/ros2_controllers.yaml</parameters>
-                <robot_param_node>/robot_state_publisher</robot_param_node>
-        </plugin>
-    </gazebo> -->
 </robot>

File: sbot_moveit/config/scorbot.urdf.xacro (robot description, xacro)
@@ -6,9 +6,5 @@
     <!-- Import control_xacro -->
     <xacro:include filename="scorbot.ros2_control.xacro" />
-    <!-- <include if="$(arg fake)"> -->
+    <!-- Macro control_xacro -->
     <xacro:scorbot_ros2_control name="FakeSystem" system="mock_components/GenericSystem"  initial_positions_file="$(arg initial_positions_file)"/>
-    <!-- </include> -->
-    <!-- <xacro:if value="$(arg sim_gz)">
-        <xacro:scorbot_ros2_control name="IgnitionSystem" system="ign_ros2_control/IgnitionSystem" initial_positions_file="$(arg initial_positions_file)"/>
-    </xacro:if>  -->
 </robot>

Commit message: Sbot_funcional

File: sbot_description/urdf/sbot_arm.urdf.xacro (robot description, xacro)
@@ -109,6 +109,6 @@
                 child="${upper_arm}"
                 limit_e="1000"
-                limit_l="-2.3562"
-                limit_u="2.3562"
+                limit_l="-2.268"
+                limit_u="0.349"
                 limit_v="0.5" />
     <xacro:m_joint name="${elbow}" type="revolute"
@@ -119,6 +119,6 @@
                 child="${forearm}"
                 limit_e="1000"
-                limit_l="-2.3562"
-                limit_u="2.3562"
+                limit_l="-0.698"
+                limit_u="3.316"
                 limit_v="0.5" />
     <xacro:m_joint name="${pitch}" type="revolute"
@@ -129,6 +129,6 @@
                 child="${flange}"
                 limit_e="1000"
-                limit_l="-2.3562"
-                limit_u="2.3562"
+                limit_l="-1.483"
+                limit_u="1.745"
                 limit_v="0.5" />
     <!-- DEFINO UN CILINDRO INTERMEDIO PARA QUE GIRE EL GRIPPER LUEGO -->
@@ -150,5 +150,5 @@
       </collision> -->
     </link>
-    <xacro:m_joint name="${roll}" type="continuous"
+    <xacro:m_joint name="${roll}" type="revolute"
                   axis_xyz="0 0 -1"
                   origin_rpy="-1.5708 0 -1.5708"
@@ -157,6 +157,6 @@
                   child="cylinder_link"
                   limit_e="1000"
-                  limit_l="-2.3562"
-                  limit_u="2.3562"
+                  limit_l="-3.1415"
+                  limit_u="3.1415"
                   limit_v="0.5" />
     <!-- DEFINO EE_LINK -->

File: sbot_description/urdf/scorbot.urdf.xacro (robot description, xacro)
@@ -16,4 +16,27 @@
         <origin xyz="0.0 0.0 0.0" rpy="0.0 0.0 0.0" />
     </joint>
+    <link name="suelo">
+      <visual>
+        <origin rpy="0 0 0" xyz="0 0 0" />
+        <geometry>
+          <cylinder radius="1" length="0.01" />
+        </geometry>
+      </visual>
+      <collision>
+            <origin rpy="0 0 0" xyz="0 0 0" />
+        <geometry>
+          <cylinder radius="1" length="0.01" />
+        </geometry>
+      </collision>
+    </link>
+    <joint name="suelo_fixed_joint" type="fixed">
+      <origin xyz="0.0 0.0 0.0" rpy="0 0 0"/>
+      <parent link="world"/>
+      <child link="suelo"/>
+    </joint>
+    <!-- For suelo -->
+  <gazebo reference="suelo">
+    <material>Gazebo/Black</material>
+  </gazebo>
     <!-- GENERAR EL GRIPPER -->
     <xacro:sbot_gripper prefix="" parent="tool0">
