Commit message: ros2_control+gazebo

File: sbot_gazebo/config/control_gazebo.xacro (robot description, xacro)
@@ -100,3 +100,30 @@
             </actuator>
         </transmission>
+    <gazebo>
+        <xacro:macro name="joint_position_controller" params="joint_name p_gain:=1 d_gain:=0 i_gain:=0 mimic_joint:=''">
+            <plugin filename="ignition-gazebo-joint-position-controller-system"
+                name="gz::sim::systems::JointPositionController">
+                <xacro:if value="${mimic_joint == ''}">
+                <xacro:property name="topic_joint" value="${joint_name}"/>
+                </xacro:if>
+                <xacro:unless value="${mimic_joint == ''}">
+                <xacro:property name="topic_joint" value="${mimic_joint}"/>
+                </xacro:unless>
+                <joint_name>${joint_name}</joint_name>
+                <p_gain>${p_gain}</p_gain>
+                <d_gain>${d_gain}</d_gain>
+                <i_gain>${i_gain}</i_gain>
+                <i_max>1000</i_max>
+                <i_min>-1000</i_min>
+                <topic>/model/scorbot/joint/${topic_joint}/cmd_pos</topic>
+            </plugin>
+        </xacro:macro>
+        <xacro:joint_position_controller joint_name="base_joint" p_gain="1e4" d_gain="1e1" i_gain="1e1"/>
+        <xacro:joint_position_controller joint_name="elbow" p_gain="1e4" d_gain="1e1" i_gain="1e1"/>
+        <xacro:joint_position_controller joint_name="shoulder" p_gain="1e4" d_gain="1e1" i_gain="1e1"/>
+        <xacro:joint_position_controller joint_name="pitch" p_gain="1e4" d_gain="1e1" i_gain="1e1"/>
+        <xacro:joint_position_controller joint_name="roll" p_gain="1e4" d_gain="1e1" i_gain="1e1"/>
+        <xacro:joint_position_controller joint_name="finger_R_joint" p_gain="1e4" d_gain="1e1" i_gain="1e1" mimic_joint="finger_L_joint"/>
+        <xacro:joint_position_controller joint_name="finger_L_joint" p_gain="1e4" d_gain="1e" i_gain="1e1"/>
+    </gazebo>
 </robot>

File: sbot_gazebo/config/sbot.urdf.xacro (robot description, xacro)
@@ -4,6 +4,8 @@
     <xacro:include filename="$(find sbot_description)/urdf/scorbot.urdf.xacro" />
     <!-- Import control_xacro -->
-    <!-- <xacro:include filename="transmission_gazebo.xacro" /> -->
-      <!-- JOINT PUBLISHER -->
+    <!-- <xacro:include filename="control_gazebo.xacro" /> -->
+    <!-- Import ignition_ros2_control conection file -->
+    <xacro:include filename="$(find sbot_gazebo)/config/gz_ros2_control.xacro" />
+          <!-- JOINT PUBLISHER -->
   <gazebo>
    <self_collide>true</self_collide>
@@ -21,29 +23,4 @@
       <joint_name>roll</joint_name>
     </plugin>
-    <xacro:macro name="joint_position_controller" params="joint_name p_gain:=1 d_gain:=0 i_gain:=0 mimic_joint:=''">
-      <plugin filename="ignition-gazebo-joint-position-controller-system"
-        name="gz::sim::systems::JointPositionController">
-        <xacro:if value="${mimic_joint == ''}">
-          <xacro:property name="topic_joint" value="${joint_name}"/>
-        </xacro:if>
-        <xacro:unless value="${mimic_joint == ''}">
-          <xacro:property name="topic_joint" value="${mimic_joint}"/>
-        </xacro:unless>
-        <joint_name>${joint_name}</joint_name>
-        <p_gain>${p_gain}</p_gain>
-        <d_gain>${d_gain}</d_gain>
-        <i_gain>${i_gain}</i_gain>
-        <i_max>1000</i_max>
-        <i_min>-1000</i_min>
-        <topic>/model/scorbot/joint/${topic_joint}/cmd_pos</topic>
-      </plugin>
-    </xacro:macro>
-    <xacro:joint_position_controller joint_name="base_joint" p_gain="1e4" d_gain="1e1" i_gain="1e1"/>
-    <xacro:joint_position_controller joint_name="elbow" p_gain="1e4" d_gain="1e1" i_gain="1e1"/>
-    <xacro:joint_position_controller joint_name="shoulder" p_gain="1e4" d_gain="1e1" i_gain="1e1"/>
-    <xacro:joint_position_controller joint_name="pitch" p_gain="1e4" d_gain="1e1" i_gain="1e1"/>
-    <xacro:joint_position_controller joint_name="roll" p_gain="1e4" d_gain="1e1" i_gain="1e1"/>
-    <xacro:joint_position_controller joint_name="finger_R_joint" p_gain="1e4" d_gain="1e1" i_gain="1e1" mimic_joint="finger_L_joint"/>
-    <xacro:joint_position_controller joint_name="finger_L_joint" p_gain="1e4" d_gain="1e" i_gain="1e1"/>
   </gazebo>
 </robot>

File: sbot_gazebo/config/scorbot.ros2_control.xacro (robot description, xacro)
@@ -1,12 +1,11 @@
 <?xml version="1.0"?>
 <robot xmlns:xacro="http://www.ros.org/wiki/xacro">
-    <xacro:macro name="sbot_ros2_control" params="name initial_positions_file">
-        <xacro:property name="initial_positions" value="${load_yaml(initial_positions_file)['initial_positions']}"/>
+    <xacro:macro name="scorbot_ros2_control" params="name initial_positions_file">
+        <xacro:property name="initial_positions" value="${xacro.load_yaml(initial_positions_file)['initial_positions']}"/>
         <ros2_control name="${name}" type="system">
             <hardware>
                 <!-- By default, set up controllers for simulation. This won't work on real hardware -->
-                <plugin>gazebo_ros_control/GazeboSystem</plugin>
-                <!-- <plugin>ign_ros2_control/IgnitionSystem</plugin> -->
                 <!-- <plugin>mock_components/GenericSystem</plugin> -->
+                <plugin>ign_ros2_control/IgnitionSystem</plugin>
             </hardware>
             <joint name="base_joint">
@@ -53,9 +52,4 @@
             </joint>
         </ros2_control>
-        <gazebo>
-          <plugin name="gazebo_ros2_control" filename="libgazebo_ros2_control.so">
-            <parameters>"$(find sbot_moveit_gz)/config/ros2_controllers.yaml"</parameters>
-          </plugin>
-        </gazebo>
     </xacro:macro>
 </robot>

File: sbot_moveit_gz/config/scorbot.ros2_control.xacro (robot description, xacro)
@@ -1,9 +1,10 @@
 <?xml version="1.0"?>
 <robot xmlns:xacro="http://www.ros.org/wiki/xacro">
-    <xacro:macro name="sbot_ros2_control" params="name initial_positions_file">
+    <xacro:macro name="scorbot_ros2_control" params="name initial_positions_file">
         <xacro:property name="initial_positions" value="${load_yaml(initial_positions_file)['initial_positions']}"/>
         <ros2_control name="${name}" type="system">
             <hardware>
                 <!-- By default, set up controllers for simulation. This won't work on real hardware -->
+                <!-- <plugin>mock_components/GenericSystem</plugin> -->
                 <plugin>ign_ros2_control/IgnitionSystem</plugin>
             </hardware>

File: sbot_moveit_gz/config/scorbot.urdf.xacro (robot description, xacro)
@@ -1,9 +1,9 @@
 <?xml version="1.0"?>
-<robot xmlns:xacro="http://www.ros.org/wiki/xacro" name="sbot">
+<robot xmlns:xacro="http://www.ros.org/wiki/xacro" name="scorbot">
     <xacro:arg name="initial_positions_file" default="initial_positions.yaml" />
-    <!-- Import sbot urdf file -->
+    <!-- Import scorbot urdf file -->
     <xacro:include filename="$(find sbot_description)/urdf/scorbot.urdf.xacro" />
     <!-- Import control_xacro -->
     <xacro:include filename="scorbot.ros2_control.xacro" />
-    <xacro:sbot_ros2_control name="FakeSystem" initial_positions_file="$(arg initial_positions_file)"/>
+    <xacro:scorbot_ros2_control name="FakeSystem" initial_positions_file="$(arg initial_positions_file)"/>
 </robot>
