Commit message: Comienzo de unión

File: sbot_gazebo/config/sbot.urdf.xacro (robot description, xacro)
@@ -4,7 +4,7 @@
     <xacro:include filename="$(find sbot_description)/urdf/scorbot.urdf.xacro" />
     <!-- Import control_xacro -->
-    <!-- <xacro:include filename="control_gazebo.xacro" /> -->
+    <xacro:include filename="control_gazebo.xacro" />
     <!-- Import ignition_ros2_control conection file -->
-    <xacro:include filename="$(find sbot_gazebo)/config/gz_ros2_control.xacro" />
+    <!-- <xacro:include filename="$(find sbot_gazebo)/config/gz_ros2_control.xacro" /> -->
           <!-- JOINT PUBLISHER -->
   <gazebo>

File: sbot_moveit/config/scorbot.ros2_control.xacro (robot description, xacro)
@@ -1,5 +1,5 @@
 <?xml version="1.0"?>
 <robot xmlns:xacro="http://www.ros.org/wiki/xacro">
-    <xacro:macro name="scorbot_ros2_control" params="name initial_positions_file">
+    <xacro:macro name="scorbot_ros2_control" params="name initial_positions_file system">
         <xacro:property name="initial_positions" value="${load_yaml(initial_positions_file)['initial_positions']}"/>
         <ros2_control name="${name}" type="system">

File: sbot_moveit/config/scorbot.urdf.xacro (robot description, xacro)
@@ -1,16 +1,17 @@
 <?xml version="1.0"?>
 <robot xmlns:xacro="http://www.ros.org/wiki/xacro" name="scorbot">
-    <arg name="sim_gazebo"            default="False"/>
-    <arg name="no_sim_gazebo"         default="True"/>
+    <!-- <arg name="sim_gazebo"            default="False"/>
+    <arg name="no_sim_gazebo"         default="True"/> -->
     <xacro:arg name="initial_positions_file" default="initial_positions.yaml" />
     <!-- Import scorbot urdf file -->
     <xacro:include filename="$(find sbot_description)/urdf/scorbot.urdf.xacro" />
     <xacro:include filename="scorbot.ros2_control.xacro" />
-    <include if="$(arg sim_gazebo)">
+    <!-- <include if="$(arg sim_gazebo)">
         <xacro:scorbot_ros2_control name="IgnSystem"
         system="ign_ros2_control/IgnitionSystem"
         initial_positions_file="$(arg initial_positions_file)"/>
-    </include>
-    <include if="$(arg no_sim_gazebo)">
+    </include> -->
+    <!-- <include if="$(arg no_sim_gazebo)"> -->
+     <include>
         <!-- Import control_xacro -->
         <xacro:scorbot_ros2_control name="FakeSystem"
